File: EAGLE/IDS_ADC.brd (EAGLE design)
At the start: 71.4 x 62.9 mm, 17 parts, among them IC1 NE5532N, IC2 NE5532N

Commit message: Add files via upload
Parts:
- removed R7: (no value), pot:RJ9W
- added R4: 10k, rcl:0207/7
- C1: value (none) -> 10u; device rcl:E5-8,5 -> rcl:E2,5-7
- C2: value (none) -> 1n
- IC1, IC2: value NE5532N -> (none)
- R1, R3: value (none) -> 10k
- R2: value (none) -> 3k
- R5: value (none) -> 10k; device rcl:0207/7 -> pot:RJ9W
- moved R5 10.2 mm to (59.7, 32.7), turned to 0 degrees
Connections:
- net ADC-IN: now also R4.2; no longer R5.2
- net GND: now also R4.1, R5.A; no longer R5.1, R7.A
- net N$15: now also R5.E; no longer R7.E
- net N$8: now also R5.S; no longer R7.S
Routing:
- net N$8: track 33.1 -> 34.4 mm
Changed lines of the file:
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@@
 HvA
 Voswijk, Hupkens, Berg</text>
+<dimension x1="3.81" y1="-1.5875" x2="75.235" y2="-1.5875" x3="39.5225" y3="-3.4925" textsize="1.778" layer="27"/>
+<dimension x1="75.235" y1="-1.5875" x2="75.235" y2="61.2675" x3="81.5975" y3="29.84" textsize="1.778" layer="27"/>
 </plain>
 <attributes>
@@
 <attribute name="VALUE" x="30.48" y="36.449" size="1.27" layer="28" ratio="10" rot="MR270"/>
 </element>
-<element name="IC1" library="linear" library_urn="urn:adsk.eagle:library:262" package="DIL08" package3d_urn="urn:adsk.eagle:package:16409/2" value="NE5532N" x="45.72" y="40.64" smashed="yes" rot="MR0">
+<element name="IC1" library="linear" library_urn="urn:adsk.eagle:library:262" package="DIL08" package3d_urn="urn:adsk.eagle:package:16409/2" value="" x="45.72" y="40.64" smashed="yes" rot="MR0">
 <attribute name="NAME" x="51.054" y="37.719" size="1.27" layer="26" ratio="10" rot="MR90"/>
 <attribute name="POPULARITY" value="0" x="45.72" y="40.64" size="1.778" layer="28" rot="MR0" display="off"/>
 <attribute name="VALUE" x="49.276" y="40.005" size="1.27" layer="28" ratio="10" rot="MR0"/>
 </element>
-<element name="IC2" library="linear" library_urn="urn:adsk.eagle:library:262" package="DIL08" package3d_urn="urn:adsk.eagle:package:16409/2" value="NE5532N" x="45.72" y="17.78" smashed="yes" rot="MR0">
+<element name="IC2" library="linear" library_urn="urn:adsk.eagle:library:262" package="DIL08" package3d_urn="urn:adsk.eagle:package:16409/2" value="" x="45.72" y="17.78" smashed="yes" rot="MR0">
 <attribute name="NAME" x="51.054" y="14.859" size="1.27" layer="26" ratio="10" rot="MR90"/>
 <attribute name="POPULARITY" value="0" x="45.72" y="17.78" size="1.778" layer="28" rot="MR0" display="off"/>
 <attribute name="VALUE" x="49.276" y="17.145" size="1.27" layer="28" ratio="10" rot="MR0"/>
 </element>
-<element name="R1" library="rcl" library_urn="urn:adsk.eagle:library:334" package="0207/7" package3d_urn="urn:adsk.eagle:package:23493/2" value="" x="42.2275" y="30.7975" smashed="yes" rot="R270">
+<element name="R1" library="rcl" library_urn="urn:adsk.eagle:library:334" package="0207/7" package3d_urn="urn:adsk.eagle:package:23493/2" value="10k" x="42.2275" y="30.7975" smashed="yes" rot="R270">
 <attribute name="NAME" x="43.6245" y="33.3375" size="1.27" layer="25" ratio="10" rot="R270"/>
 <attribute name="POPULARITY" value="46" x="42.2275" y="30.7975" size="1.778" layer="27" rot="R270" display="off"/>
@@
 <attribute name="VALUE" x="41.6687" y="33.0835" size="1.27" layer="27" ratio="10" rot="R270"/>
 </element>
-<element name="R2" library="rcl" library_urn="urn:adsk.eagle:library:334" package="0207/7" package3d_urn="urn:adsk.eagle:package:23493/2" value="" x="49.2125" y="26.3525" smashed="yes">
+<element name="R2" library="rcl" library_urn="urn:adsk.eagle:library:334" package="0207/7" package3d_urn="urn:adsk.eagle:package:23493/2" value="3k" x="49.2125" y="26.3525" smashed="yes">
 <attribute name="NAME" x="46.6725" y="27.7495" size="1.27" layer="25" ratio="10"/>
 <attribute name="POPULARITY" value="46" x="49.2125" y="26.3525" size="1.778" layer="27" display="off"/>
@@
 <attribute name="VALUE" x="46.9265" y="25.7937" size="1.27" layer="27" ratio="10"/>
 </element>
-<element name="R5" library="rcl" library_urn="urn:adsk.eagle:library:334" package="0207/7" package3d_urn="urn:adsk.eagle:package:23493/2" value="" x="53.34" y="40.64" smashed="yes" rot="R270">
+<element name="R4" library="rcl" library_urn="urn:adsk.eagle:library:334" package="0207/7" package3d_urn="urn:adsk.eagle:package:23493/2" value="10k" x="53.34" y="40.64" smashed="yes" rot="R270">
 <attribute name="NAME" x="54.737" y="43.18" size="1.27" layer="25" ratio="10" rot="R270"/>
 <attribute name="POPULARITY" value="46" x="53.34" y="40.64" size="1.778" layer="27" rot="R270" display="off"/>
@@
 <attribute name="VALUE" x="52.7812" y="42.926" size="1.27" layer="27" ratio="10" rot="R270"/>
 </element>
-<element name="C1" library="rcl" library_urn="urn:adsk.eagle:library:334" package="E5-8,5" package3d_urn="urn:adsk.eagle:package:23374/1" value="" x="56.1975" y="21.9075" smashed="yes" rot="R270">
+<element name="C1" library="rcl" library_urn="urn:adsk.eagle:library:334" package="E2,5-7" package3d_urn="urn:adsk.eagle:package:23345/1" value="10u" x="56.1975" y="21.9075" smashed="yes" rot="R270">
 <attribute name="NAME" x="58.4835" y="17.7673" size="1.27" layer="25" ratio="10" rot="R270"/>
-<attribute name="POPULARITY" value="0" x="56.1975" y="21.9075" size="1.778" layer="27" rot="R270" display="off"/>
+<attribute name="POPULARITY" value="17" x="56.1975" y="21.9075" size="1.778" layer="27" rot="R270" display="off"/>
 <attribute name="SPICEPREFIX" value="C" x="56.1975" y="21.9075" size="1.778" layer="27" rot="R270" display="off"/>
 <attribute name="VALUE" x="53.1749" y="24.4221" size="1.27" layer="27" ratio="10" rot="R270"/>
 </element>
-<element name="C2" library="rcl" library_urn="urn:adsk.eagle:library:334" package="C1206" package3d_urn="urn:adsk.eagle:package:23618/2" value="" x="46.355" y="29.21" smashed="yes">
+<element name="C2" library="rcl" library_urn="urn:adsk.eagle:library:334" package="C1206" package3d_urn="urn:adsk.eagle:package:23618/2" value="1n" x="46.355" y="29.21" smashed="yes">
 <attribute name="NAME" x="45.085" y="30.48" size="1.27" layer="25"/>
 <attribute name="POPULARITY" value="54" x="46.355" y="29.21" size="1.778" layer="27" display="off"/>
@@
 <attribute name="VALUE" x="46.99" y="46.355" size="1.27" layer="28" rot="MR0"/>
 </element>
-<element name="R7" library="pot" library_urn="urn:adsk.eagle:library:331" package="RJ9W" package3d_urn="urn:adsk.eagle:package:22702/1" value="" x="59.69" y="32.7025" smashed="yes">
+<element name="R5" library="pot" library_urn="urn:adsk.eagle:library:331" package="RJ9W" package3d_urn="urn:adsk.eagle:package:22702/1" value="10k" x="59.69" y="32.7025" smashed="yes">
 <attribute name="NAME" x="55.118" y="35.3695" size="1.27" layer="25" ratio="10"/>
 <attribute name="POPULARITY" value="2" x="59.69" y="32.7025" size="1.778" layer="27" display="off"/>
@@
 <attribute name="VALUE" x="66.3575" y="25.781" size="1.27" layer="28" ratio="10" rot="MR270"/>
 </element>
-<element name="R3" library="rcl" library_urn="urn:adsk.eagle:library:334" package="0207/7" package3d_urn="urn:adsk.eagle:package:23493/2" value="" x="49.2125" y="33.655" smashed="yes" rot="R180">
+<element name="R3" library="rcl" library_urn="urn:adsk.eagle:library:334" package="0207/7" package3d_urn="urn:adsk.eagle:package:23493/2" value="10k" x="49.2125" y="33.655" smashed="yes" rot="R180">
 <attribute name="NAME" x="51.7525" y="32.258" size="1.27" layer="25" ratio="10" rot="R180"/>
 <attribute name="POPULARITY" value="46" x="49.2125" y="33.655" size="1.778" layer="27" rot="R180" display="off"/>
@@
 <contactref element="U$2" pad="P$20"/>
 <contactref element="U$2" pad="P$21"/>
-<contactref element="R5" pad="1"/>
+<contactref element="R4" pad="1"/>
 <contactref element="JP1" pad="2"/>
 <contactref element="U$1" pad="12"/>
@@
 <contactref element="U$4" pad="P$4"/>
 <contactref element="U$4" pad="P$1"/>
-<contactref element="R7" pad="A"/>
+<contactref element="R5" pad="A"/>
 <contactref element="U$3" pad="4"/>
 <contactref element="U$3" pad="3"/>
@@
 <contactref element="IC1" pad="2"/>
 <contactref element="IC1" pad="1"/>
-<contactref element="R5" pad="2"/>
+<contactref element="R4" pad="2"/>
 <wire x1="46.99" y1="36.83" x2="49.53" y2="36.83" width="0.508" layer="1"/>
 <wire x1="53.34" y1="36.83" x2="49.53" y2="36.83" width="0.508" layer="1"/>
@@
 <contactref element="C1" pad="+"/>
 <wire x1="50.8" y1="20.32" x2="44.45" y2="13.97" width="0.508" layer="1"/>
-<contactref element="R7" pad="S"/>
+<contactref element="R5" pad="S"/>
 <wire x1="51.1175" y1="20.6375" x2="50.8" y2="20.32" width="0.4064" layer="1"/>
 <wire x1="51.1175" y1="27.305" x2="51.1175" y2="20.6375" width="0.4064" layer="1"/>
 <wire x1="53.6575" y1="28.575" x2="56.1975" y2="26.035" width="0.4064" layer="1"/>
-<wire x1="56.1975" y1="26.035" x2="56.1975" y2="24.4475" width="0.4064" layer="1"/>
+<wire x1="56.1975" y1="26.035" x2="56.1975" y2="23.1775" width="0.4064" layer="1"/>
 <wire x1="59.69" y1="33.3375" x2="59.69" y2="29.5275" width="0.4064" layer="1"/>
 <wire x1="59.69" y1="29.5275" x2="56.1975" y2="26.035" width="0.4064" layer="1"/>
@@
 </signal>
 <signal name="N$15">
-<contactref element="R7" pad="E"/>
+<contactref element="R5" pad="E"/>
 <contactref element="R3" pad="1"/>
 <wire x1="53.0225" y1="33.655" x2="56.8325" y2="33.655" width="0.4064" layer="1"/>
